File: hive13-light-pcb.kicad_pcb (KiCad board)
At the start: 2 copper layers, 228.6 x 47.6 mm, 48 parts, among them J1 Conn_01x01_Male, J10 Conn_01x01_Male, J2 Conn_01x01_Male, J3 Conn_01x01_Male, J4 Conn_01x01_Male, J5 Conn_01x01_Male, J6 Conn_01x01_Male, J7 Conn_01x01_Male, J8 Conn_01x01_Male, J9 Conn_01x01_Male, U1 MOC3011M, U2 MOC3011M, U3 MOC3011M, U4 MOC3011M, U5 4N25, U6 WeMos_mini, U7 DS18B20

Commit message: First drawing of the PCB.
Parts:
- J1, J10, J2, J3, J4, J5, J6, J7, J8, J9: footprint Connector_Wire:SolderWirePad_1x02_P7.62mm_Drill2.5mm -> 250-Tab:250 Tab
- moved J1 32.4 mm to (174.0, 32.4)
- moved C1 28.6 mm to (170.2, 47.0)
- moved R9 28.6 mm to (180.3, 53.3)
- moved J5 27.5 mm to (114.3, 31.8)
- moved J10 20.4 mm to (140.3, 44.5)
- moved J9 14.2 mm to (126.4, 39.4), turned to 0 degrees
- moved J3 13.4 mm to (212.1, 32.4)
- moved J4 13.4 mm to (231.1, 32.4)
- moved C3 9.53 mm to (208.3, 47.0)
- moved C5 9.53 mm to (80.6, 60.3)
- moved D1 9.53 mm to (171.4, 40.6)
- moved D2 9.53 mm to (190.5, 40.6)
- moved D4 9.53 mm to (228.6, 40.6)
- moved D5 9.53 mm to (100.3, 50.8)
- moved F1 9.53 mm to (141.0, 30.5)
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Connections:
- C1 pad 1: /SNUB_2 -> /SNUB_1
- C1 pad 2: /OUT_2 -> /OUT_1
- C2 pad 1: /SNUB_1 -> /SNUB_2
- C2 pad 2: /OUT_1 -> /OUT_2
- D1 pad 2: /OUT_2 -> /OUT_1
- D1 pad 3: /GATE_2 -> /GATE_1
- D2 pad 2: /OUT_1 -> /OUT_2
- D2 pad 3: /GATE_1 -> /GATE_2
- J1 pad 1: /OUT_2 -> /OUT_1
- J2 pad 1: /OUT_1 -> /OUT_2
- R1 pad 1: /TRIAC_2 -> /TRIAC_1
- R10 pad 2: /SNUB_1 -> /SNUB_2
- R2 pad 1: /TRIAC_1 -> /TRIAC_2
- R5 pad 2: /OGATE_2 -> /OGATE_1
- R6 pad 2: /OGATE_1 -> /OGATE_2
- R9 pad 2: /SNUB_2 -> /SNUB_1
- U1 pad 4: /GATE_2 -> /GATE_1
- U1 pad 6: /OGATE_2 -> /OGATE_1
- U2 pad 4: /GATE_1 -> /GATE_2
- U2 pad 6: /OGATE_1 -> /OGATE_2
Routing:
- net /FUSED_AC: track 0.00 -> 80.0 mm
- net /NEUTRAL: track 0.00 -> 38.6 mm
- net /OUT_4: track 0.00 -> 21.2 mm
- net /OUT_2: track 0.00 -> 21.2 mm
- net /OUT_1: track 0.00 -> 21.2 mm
- net /OUT_3: track 0.00 -> 21.2 mm
- net Net-(R4-Pad2): track 138.9 -> 129.7 mm
- net /TRIAC_1: track 82.8 -> 74.5 mm
- net Net-(R2-Pad2): track 79.1 -> 85.5 mm
- net Net-(R3-Pad2): track 111.2 -> 114.5 mm
- net /TRIAC_2: track 57.8 -> 60.5 mm
- net GND: track 298.7 -> 299.9 mm
- net Net-(R1-Pad2): track 56.8 -> 57.8 mm
- net /ZCD: track 140.3 -> 141.1 mm
- added copper zone on B.Cu, net /AC
- added copper zone on F.Cu, net /AC
- added copper zone on B.Cu, net /FUSED_AC
- added copper zone on F.Cu, net /FUSED_AC
- added copper zone on B.Cu, net /NEUTRAL
- added copper zone on F.Cu, net /NEUTRAL
Other:
- board text added: "Hive13 Light Controller Board Version 1.0 (c) 2018 Greg J Arnold"
